File: MRC-RJ45-CMRI.sch (EAGLE design)
At the start: 4 parts

Commit message: moving file around
moving existing files into Github
Parts:
- removed BOARD1: BOARD80X100, SPCoast:BOARD80X100
- removed FID1, FID2: FIDUCIAL, SPCoast:FIDUCIAL
- removed OSHW1: DOC-OSHW-LOGO-M, SPCoast:DOC-OSHW-LOGO-M
- added CON1: (no value), SPCoast:CONNECTOR-M08LOCK
- added J1: (no value), con-amp:215877-7
- added J2: (no value), SparkFun:M083.5MM-8
- added J3: (no value), con-molex:KK-156-8
- added JP1, JP2: (no value), SparkFun:M023.5MM_LOCK
- added U$1: OSHW-LOGOM, SparkFun:OSHW-LOGOM
Connections:
- new net GND: JP1.1, JP1.2, JP2.1, JP2.2
- new net L1: CON1.1, J1.1, J2.1, J3-1.S
- new net L2: CON1.2, J1.2, J2.2, J3-2.S
- new net L3: CON1.3, J1.3, J2.3, J3-3.S
- new net L4: CON1.4, J1.4, J2.4, J3-4.S
- new net L5: CON1.5, J1.5, J2.5, J3-5.S
- new net L6: CON1.6, J1.6, J2.6, J3-6.S
- new net L7: CON1.7, J1.7, J2.7, J3-7.S
- new net L8: CON1.8, J1.8, J2.8, J3-8.S
Other:
- note added: "3.5mm 8-pin"
- note added: "Additional tie points"
- note added: "CMRI Breakout"
- note added: "Molex 8-pin"
- note added: "RJ45"
- note added: "RJ45 adapter"
- note added: "v2.0"
- note removed: "1.0"
- note removed: "A"
- note removed: "A Template for Eagle Projects"
- note removed: "Your Name"
